File: Hardware/Quango_Components.kicad_sch (KiCad schematic)
At the start: 112 parts, among them J1 Conn_01x12_Male, J2 Conn_01x12_Male, J3 Conn_01x12_Male, J4 Conn_01x12_Male, J5 SWD_Header, J6 Eurorack_10_pin_power, Q1 MMBT3904, U1 LM1117-3.3, U2 STM32G473V, U3 LM1117-5.0, U4 PS508, U5 MCP6002, U6 AS3364, U7 AS3364, U8 AD5676, U9 MCP48CMB21, Y1 8MHz 20pF

Commit message: Further Layout
Connections:
- net Audio1_Out: now also J2.4 (Pin_4); no longer J1.9 (Pin_9)
- net Audio2_Out: now also J2.1 (Pin_1); no longer J1.10 (Pin_10)
- net Audio3_Out: now also J2.2 (Pin_2); no longer J1.11 (Pin_11)
- net Audio4_Out: now also J2.3 (Pin_3); no longer J1.12 (Pin_12)
- net AudioA1_In: now also J1.1 (Pin_1); no longer J2.1 (Pin_1)
- net AudioA2_In: now also J1.2 (Pin_2); no longer J2.2 (Pin_2)
- net AudioA3_In: now also J1.3 (Pin_3); no longer J2.3 (Pin_3)
- net AudioA4_In: now also J1.4 (Pin_4); no longer J2.4 (Pin_4)
- net Env1_Attack: now also J1.5 (Pin_5); no longer J1.1 (Pin_1)
- net Env1_Decay: now also J1.6 (Pin_6); no longer J1.2 (Pin_2)
- net Env1_Release: now also J1.8 (Pin_8); no longer J1.4 (Pin_4)
- net Env1_Sustain: now also J1.7 (Pin_7); no longer J1.3 (Pin_3)
- net Env2_Attack: now also J1.9 (Pin_9); no longer J1.5 (Pin_5)
- net Env2_Decay: now also J1.10 (Pin_10); no longer J1.6 (Pin_6)
- net Env2_Release: now also J1.12 (Pin_12); no longer J1.8 (Pin_8)
- net Env2_Sustain: now also J1.11 (Pin_11); no longer J1.7 (Pin_7)
- net EnvA1_DAC: now also U2.26 (PA4); no longer U2.22 (PA2)
- net EnvA1_LED_Out: now also J3.7 (Pin_7); no longer J3.1 (Pin_1)
- net EnvA2_DAC: now also U2.22 (PA2); no longer U2.26 (PA4)
- net EnvA2_LED_Out: now also J3.6 (Pin_6); no longer J3.2 (Pin_2)
- net EnvA3_DAC: now also U2.28 (PA6); no longer U2.27 (PA5)
- net EnvA3_LED_Out: now also J3.8 (Pin_8); no longer J3.3 (Pin_3)
- net EnvA4_DAC: now also U2.27 (PA5); no longer U2.28 (PA6)
- net EnvA4_LED_Out: now also J3.5 (Pin_5); no longer J3.4 (Pin_4)
- net EnvB1_LED_Out: now also J3.4 (Pin_4); no longer J3.5 (Pin_5)
- net EnvB2_LED_Out: now also J3.3 (Pin_3); no longer J3.6 (Pin_6)
- net EnvB3_LED_Out: now also J3.2 (Pin_2); no longer J3.7 (Pin_7)
- net EnvB4_LED_Out: now also J3.1 (Pin_1); no longer J3.8 (Pin_8)
Changed lines of the file:
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@@
     (effects (font (size 1.27 1.27)) (justify right bottom))
   )
-  (label "AudioA4_In" (at -203.2 -35.56 0)
+  (label "AudioA4_In" (at -203.2 -74.93 0)
     (effects (font (size 1.27 1.27)) (justify left bottom))
   )
@@
     (effects (font (size 1.27 1.27)) (justify left bottom))
   )
-  (label "EnvA1_DAC" (at 99.06 48.26 0)
+  (label "EnvA1_DAC" (at 99.06 53.34 0)
     (effects (font (size 1.27 1.27)) (justify left bottom))
   )
@@
     (effects (font (size 1.27 1.27)) (justify left bottom))
   )
-  (label "EnvA4_DAC" (at 99.06 58.42 0)
+  (label "EnvA4_DAC" (at 99.06 55.88 0)
     (effects (font (size 1.27 1.27)) (justify left bottom))
   )
@@
     (effects (font (size 1.27 1.27)) (justify left bottom))
   )
-  (label "EnvA3_LED_Out" (at -175.26 -78.74 0)
+  (label "EnvA3_LED_Out" (at -175.26 -66.04 0)
     (effects (font (size 1.27 1.27)) (justify left bottom))
   )
@@
     (effects (font (size 1.27 1.27)) (justify left bottom))
   )
-  (label "Audio2_Out" (at -203.2 -59.69 0)
+  (label "Audio2_Out" (at -203.2 -43.18 0)
     (effects (font (size 1.27 1.27)) (justify left bottom))
   )
@@
     (effects (font (size 1.27 1.27)) (justify right bottom))
   )
-  (label "EnvB4_LED_Out" (at -175.26 -66.04 0)
+  (label "EnvB4_LED_Out" (at -175.26 -83.82 0)
     (effects (font (size 1.27 1.27)) (justify left bottom))
   )
@@
     (effects (font (size 1.27 1.27)) (justify left bottom))
   )
-  (label "EnvA3_DAC" (at 99.06 55.88 0)
+  (label "EnvA3_DAC" (at 99.06 58.42 0)
     (effects (font (size 1.27 1.27)) (justify left bottom))
   )
@@
     (effects (font (size 1.27 1.27)) (justify right bottom))
   )
-  (label "AudioA2_In" (at -203.2 -40.64 0)
+  (label "AudioA2_In" (at -203.2 -80.01 0)
     (effects (font (size 1.27 1.27)) (justify left bottom))
   )
@@
     (effects (font (size 1.27 1.27)) (justify left bottom))
   )
-  (label "Audio4_Out" (at -203.2 -54.61 0)
-    (effects (font (size 1.27 1.27)) (justify left bottom))
-  )
-  (label "AudioA1_In" (at -203.2 -43.18 0)
+  (label "Audio4_Out" (at -203.2 -38.1 0)
+    (effects (font (size 1.27 1.27)) (justify left bottom))
+  )
+  (label "AudioA1_In" (at -203.2 -82.55 0)
     (effects (font (size 1.27 1.27)) (justify left bottom))
   )
@@
     (effects (font (size 1.27 1.27)) (justify right bottom))
   )
-  (label "Env2_Decay" (at -203.2 -69.85 0)
+  (label "Env2_Decay" (at -203.2 -59.69 0)
     (effects (font (size 1.27 1.27)) (justify left bottom))
   )
@@
     (effects (font (size 1.27 1.27)) (justify right bottom))
   )
-  (label "Env2_Release" (at -203.2 -64.77 0)
+  (label "Env2_Release" (at -203.2 -54.61 0)
     (effects (font (size 1.27 1.27)) (justify left bottom))
   )
@@
     (effects (font (size 1.27 1.27)) (justify left bottom))
   )
-  (label "EnvB2_LED_Out" (at -175.26 -71.12 0)
+  (label "EnvB2_LED_Out" (at -175.26 -78.74 0)
     (effects (font (size 1.27 1.27)) (justify left bottom))
   )
@@
     (effects (font (size 1.27 1.27)) (justify right bottom))
   )
-  (label "Env2_Sustain" (at -203.2 -67.31 0)
+  (label "Env2_Sustain" (at -203.2 -57.15 0)
     (effects (font (size 1.27 1.27)) (justify left bottom))
   )
@@
     (effects (font (size 1.27 1.27)) (justify right bottom))
   )
-  (label "EnvA2_DAC" (at 99.06 53.34 0)
+  (label "EnvA2_DAC" (at 99.06 48.26 0)
     (effects (font (size 1.27 1.27)) (justify left bottom))
   )
@@
     (effects (font (size 1.27 1.27)) (justify left bottom))
   )
-  (label "EnvB3_LED_Out" (at -175.26 -68.58 0)
+  (label "EnvB3_LED_Out" (at -175.26 -81.28 0)
     (effects (font (size 1.27 1.27)) (justify left bottom))
   )
@@
     (effects (font (size 1.27 1.27)) (justify left bottom))
   )
-  (label "Env1_Sustain" (at -203.2 -77.47 0)
+  (label "Env1_Sustain" (at -203.2 -67.31 0)
     (effects (font (size 1.27 1.27)) (justify left bottom))
   )
@@
     (effects (font (size 1.27 1.27)) (justify left bottom))
   )
-  (label "Env1_Attack" (at -203.2 -82.55 0)
+  (label "Env1_Attack" (at -203.2 -72.39 0)
     (effects (font (size 1.27 1.27)) (justify left bottom))
   )
@@
     (effects (font (size 1.27 1.27)) (justify right bottom))
   )
-  (label "Env2_Attack" (at -203.2 -72.39 0)
+  (label "Env2_Attack" (at -203.2 -62.23 0)
     (effects (font (size 1.27 1.27)) (justify left bottom))
   )
@@
     (effects (font (size 1.27 1.27)) (justify left bottom))
   )
-  (label "Audio3_Out" (at -203.2 -57.15 0)
+  (label "Audio3_Out" (at -203.2 -40.64 0)
     (effects (font (size 1.27 1.27)) (justify left bottom))
   )
@@
     (effects (font (size 1.27 1.27)) (justify right bottom))
   )
-  (label "EnvA1_LED_Out" (at -175.26 -83.82 0)
+  (label "EnvA1_LED_Out" (at -175.26 -68.58 0)
     (effects (font (size 1.27 1.27)) (justify left bottom))
   )
@@
     (effects (font (size 1.27 1.27)) (justify right bottom))
   )
-  (label "EnvB1_LED_Out" (at -175.26 -73.66 0)
+  (label "EnvB1_LED_Out" (at -175.26 -76.2 0)
     (effects (font (size 1.27 1.27)) (justify left bottom))
   )
@@
     (effects (font (size 1.27 1.27)) (justify left bottom))
   )
-  (label "Env1_Decay" (at -203.2 -80.01 0)
+  (label "Env1_Decay" (at -203.2 -69.85 0)
     (effects (font (size 1.27 1.27)) (justify left bottom))
   )
@@
     (effects (font (size 1.27 1.27)) (justify left bottom))
   )
-  (label "Env1_Release" (at -203.2 -74.93 0)
+  (label "Env1_Release" (at -203.2 -64.77 0)
     (effects (font (size 1.27 1.27)) (justify left bottom))
   )
@@
     (effects (font (size 1.27 1.27)) (justify left bottom))
   )
-  (label "AudioA3_In" (at -203.2 -38.1 0)
+  (label "AudioA3_In" (at -203.2 -77.47 0)
     (effects (font (size 1.27 1.27)) (justify left bottom))
   )
@@
     (effects (font (size 1.27 1.27)) (justify right bottom))
   )
-  (label "EnvA4_LED_Out" (at -175.26 -76.2 0)
+  (label "EnvA4_LED_Out" (at -175.26 -73.66 0)
     (effects (font (size 1.27 1.27)) (justify left bottom))
   )
@@
     (effects (font (size 1.27 1.27)) (justify left bottom))
   )
-  (label "EnvA2_LED_Out" (at -175.26 -81.28 0)
+  (label "EnvA2_LED_Out" (at -175.26 -71.12 0)
     (effects (font (size 1.27 1.27)) (justify left bottom))
   )
@@
     (effects (font (size 1.27 1.27)) (justify right bottom))
   )
-  (label "Audio1_Out" (at -203.2 -62.23 0)
-    (effects (font (size 1.27 1.27)) (justify left bottom))
-  )
+  (label "Audio1_Out" (at -203.2 -35.56 0)
+    (effects (font (size 1.27 1.27)) (justify left bottom))
+  )
